File: RC-W25/RC_Battery.kicad_sch (KiCad schematic)
At the start: 18 parts, among them P2 CONN HEADER SMD R/A 2POS 2MM, SW1 JS202011JAQN, U2 AP62300TWU, U5 MCP73831-5-OT

Commit message: Almost Finalized Schematic
Still need to spec out buttons and jst conn
Parts:
- removed P2: CONN HEADER SMD R/A 2POS 2MM, Library:CONN02_502352_MOL, symbol New_Library:DuraClik_CONN_HEADER_SMD_R/A_2POS_2MM
- removed SW1: JS202011JAQN, Library:JS202011JAQN, symbol New_Library_6:JS202011JAQN
- added P1: JST CONN, Library:CONN02_502352_MOL, symbol Connector_Generic:Conn_01x02
- added SW1: Toggle Button, symbol Switch:SW_SPST
- C10: renamed from C14; footprint Capacitor_SMD:C_0603_1608Metric -> Capacitor_SMD:C_0402_1005Metric; LCSC# (none) -> C22399610
- C11: renamed from C15; footprint Capacitor_SMD:C_0603_1608Metric -> Capacitor_SMD:C_0402_1005Metric; LCSC# (none) -> C22399610
- C12: renamed from C5; LCSC# (none) -> C95839
- C13: renamed from C6; footprint Capacitor_SMD:C_0603_1608Metric -> Capacitor_SMD:C_0402_1005Metric; LCSC# (none) -> C22435938
- C14: renamed from C7; footprint Capacitor_SMD:C_0603_1608Metric -> Capacitor_SMD:C_0805_2012Metric; LCSC# (none) -> C380337
- C15: renamed from C8; footprint Capacitor_SMD:C_0603_1608Metric -> Capacitor_SMD:C_0805_2012Metric; LCSC# (none) -> C380337
- D4: renamed from D1; value LED_Small -> LED; footprint (none) -> Diode_SMD:D_0402_1005Metric; LCSC# (none) -> C7496801
- R10: renamed from R1; footprint Resistor_SMD:R_0603_1608Metric -> Resistor_SMD:R_0402_1005Metric; LCSC# (none) -> C5137149
- R11: renamed from R9; footprint Resistor_SMD:R_0603_1608Metric -> Resistor_SMD:R_0402_1005Metric; LCSC# (none) -> C190095
- R12: renamed from R7; footprint Resistor_SMD:R_0603_1608Metric -> Resistor_SMD:R_0402_1005Metric; LCSC# (none) -> C2681602
- R13: renamed from R8; footprint Resistor_SMD:R_0603_1608Metric -> Resistor_SMD:R_0402_1005Metric; LCSC# (none) -> C190095
- R8: renamed from R13; footprint Resistor_SMD:R_0603_1608Metric -> Resistor_SMD:R_0402_1005Metric; LCSC# (none) -> C852799
- R9: renamed from R12; footprint Resistor_SMD:R_0603_1608Metric -> Resistor_SMD:R_0402_1005Metric; LCSC# (none) -> C2902640
- U2: renamed from U5; footprint Package_TO_SOT_SMD:SOT-23-5 -> Package_DFN_QFN:DFN-8-1EP_2x3mm_P0.5mm_EP0.61x2.2mm; LCSC# (none) -> C635037
- U3: renamed from U2; LCSC# (none) -> C1883519
Connections:
- net +VPRE is gone; now on net +VBAT: C12.1, U3.3 (IN)
- net +VBAT: now also SW1.2 (B); no longer C11.1, R10.1, U2.3 (V_{BAT})
- net GND: now also P1.2 (Pin_2)
- net +5V renamed +USB5V
- new net: C11.1, P1.1 (Pin_1), R10.1, SW1.1 (A), U2.3 (V_{BAT})
Other:
- note added: "{dblquote}on/off switch{dblquote}"
- note removed: "Power Switch"
