File: RC-W25/RC-W25.kicad_pcb (KiCad board)
At the start: 2 copper layers, 36 x 100.1 mm, 55 parts, among them J1 USB_C_Receptacle_USB2.0_14P, P1 JST CONN, P2 JST CONN, Q1 NMOS, SW1 Button, SW2 Button, SW3 YTSPS-22E58LM, SW4 Button, U1 ESP32-C6-MINI-1, U2 MCP73831-5-OT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

Commit message: crc v1
quick fixes
Parts:
- DS1: footprint Library:FPC_30 -> footprints:FPC-30P-0.5mm
- L1: footprint Inductor_SMD:L_Abracon_ASPI-4030S -> footprints:L_Abracon_ASPI-4030S
Changed lines of the file:
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@@
 			(pintype "passive")
 		)
-		(model "C:/Users/Matthew/Downloads/3dpea.com_TS-1088-AR2016.step"
+		(model "${KIPRJMOD}/models.3dshapes/button.3dshapes/SW-SMD_L3.9-W2.9-H2.0-LS4.8.step"
 			(offset
 				(xyz 0 0 0)
 			)
 			(scale
-				(xyz 100 100 100)
+				(xyz 1 1 1)
 			)
 			(rotate
-				(xyz -90 0 0)
+				(xyz 0 0 0)
 			)
 		)
@@
 		)
 	)
-	(footprint "Inductor_SMD:L_Abracon_ASPI-4030S"
+	(footprint "footprints:L_Abracon_ASPI-4030S"
 		(layer "F.Cu")
 		(at 119.735 103 180)
@@
 		(tags "inductor abracon smd shielded")
 		(property "Reference" "L1"
-			(at 0 3 0)
+			(at 0 -3 180)
 			(layer "F.SilkS")
 			(effects
 				(font
-					(size 0.8 0.8)
-					(thickness 0.1)
+					(size 1 1)
+					(thickness 0.15)
 				)
 			)
 		)
 		(property "Value" "3.3uH"
-			(at 0 3 0)
+			(at 0 3 180)
 			(layer "F.Fab")
 			(effects
@@
 			)
 		)
-		(property "Footprint" "Inductor_SMD:L_Abracon_ASPI-4030S"
+		(property "Footprint" "footprints:L_Abracon_ASPI-4030S"
 			(at 0 0 180)
 			(unlocked yes)
@@
 		)
 		(fp_text user "${REFERENCE}"
-			(at 0 0 0)
+			(at 0 0 180)
 			(layer "F.Fab")
 			(effects
@@
 			(pintype "passive")
 		)
-		(model "${KICAD8_3DMODEL_DIR}/Inductor_SMD.3dshapes/L_Abracon_ASPI-4030S.wrl"
+		(model "${KIPRJMOD}/models.3dshapes/IND-SMD_L4.0-W4.0-H2.6_FNR40XXS.step"
 			(offset
 				(xyz 0 0 0)
@@
 		(fp_poly
 			(pts
-				(xy -1.909622 -1.27573) (xy -2.149622 -1.60573) (xy -1.669622 -1.60573) (xy -1.909622 -1.27573)
+				(xy -1.3 -1.51) (xy -1.54 -1.84) (xy -1.06 -1.84) (xy -1.3 -1.51)
 			)
 			(stroke
@@
 			(pintype "passive")
 		)
-		(model "C:/Users/Matthew/Downloads/3dpea.com_TS-1088-AR2016.step"
+		(model "${KIPRJMOD}/models.3dshapes/button.3dshapes/SW-SMD_L3.9-W2.9-H2.0-LS4.8.step"
 			(offset
 				(xyz 0 0 0)
 			)
 			(scale
-				(xyz 100 100 100)
+				(xyz 1 1 1)
 			)
 			(rotate
-				(xyz -90 0 0)
+				(xyz 0 0 0)
 			)
 		)
@@
 			(layers "F.Cu" "F.Paste" "F.Mask")
 		)
+		(model "${KIPRJMOD}/models.3dshapes/CONN-SMD_2P-P2.00_XUNPU_WAFER-PH2.0-2PWB.step"
+			(offset
+				(xyz 0 1.5 2.7)
+			)
+			(scale
+				(xyz 1 1 1)
+			)
+			(rotate
+				(xyz 0 0 0)
+			)
+		)
 	)
 	(footprint "Diode_SMD:D_0402_1005Metric"
@@
 		)
 	)
-	(footprint "Library:FPC_30"
+	(footprint "footprints:FPC-30P-0.5mm"
 		(layer "F.Cu")
 		(at 125.002844 74.674494)
@@
 			(effects
 				(font
-					(size 0.8 0.8)
-					(thickness 0.1)
+					(size 1 1)
+					(thickness 0.15)
 				)
 			)
@@
 			)
 		)
-		(property "Footprint" "Library:FPC_30"
+		(property "Footprint" "footprints:FPC-30P-0.5mm"
 			(at 0 0 0)
 			(layer "F.Fab")
@@
 			(thermal_bridge_angle 45)
 		)
-		(model "${KICAD8_3DMODEL_DIR}/Resistor_SMD.3dshapes/R_0201_0603Metric.step"
+		(model "${KIPRJMOD}/models.3dshapes/fpc30p.3dshapes/FPC-SMD_30P-P0.50_XUNPU_FPC-05F-30PH20.step"
 			(offset
-				(xyz 0 -2 0)
+				(xyz 0 0.5 0)
 			)
 			(scale
-				(xyz 32 15 6)
+				(xyz 1 1 1)
 			)
 			(rotate
@@
 			(layers "F.Cu" "F.Paste" "F.Mask")
 		)
+		(model "${KIPRJMOD}/models.3dshapes/CONN-SMD_2P-P2.00_XUNPU_WAFER-PH2.0-2PWB.step"
+			(offset
+				(xyz 0 1.5 2.7)
+			)
+			(scale
+				(xyz 1 1 1)
+			)
+			(rotate
+				(xyz 0 0 0)
+			)
+		)
 	)
 	(footprint "Resistor_SMD:R_0402_1005Metric"
@@
 		(fp_arc
 			(start 0.3048 -0.5715)
-			(mid 0 -0.266695)
+			(mid 0 -0.266698)
 			(end -0.3048 -0.5715)
 			(stroke
@@
 			(pintype "passive")
 		)
-		(model "C:/Users/Matthew/Downloads/3dpea.com_TS-1088-AR2016.step"
+		(model "${KIPRJMOD}/models.3dshapes/button.3dshapes/SW-SMD_L3.9-W2.9-H2.0-LS4.8.step"
 			(offset
 				(xyz 0 0 0)
 			)
 			(scale
-				(xyz 100 100 100)
+				(xyz 1 1 1)
 			)
 			(rotate
-				(xyz -90 0 0)
+				(xyz 0 0 0)
 			)
 		)
@@
 		(fp_line
 			(start 6.75 -5.75)
-			(end 6.75 5.6)
+			(end 6.75 11.15)
 			(stroke
 				(width 0.12)
@@
 		)
 		(fp_line
-			(start 6.75 5.6)
-			(end -6.75 5.6)
+			(start 6.75 11.15)
+			(end -6.75 11.15)
 			(stroke
 				(width 0.12)
@@
 		)
 		(fp_line
-			(start -6.75 5.6)
+			(start -6.75 11.15)
 			(end -6.75 -5.75)
 			(stroke

Commit message: crc v2
finalizing receiver layout
Parts:
- moved P2 1.17 mm to (118.4, 119.8), turned to -90 degrees
Routing:
- net Net-(D5-A): track 6.08 -> 13.4 mm
- net +VBAT: track 41.7 -> 43.9 mm
- net GPIO_MODE: track 42.6 -> 43.7 mm
- net GND: track 15.5 -> 14.4 mm, vias 255 -> 259
- net +3.3V: track 180.3 -> 181.1 mm
- net /RC_Connections/RESET: track 33.2 -> 34.0 mm
