File: RC-W25/RC_Connections.kicad_sch (KiCad schematic)
At the start: 28 parts, among them J1 USB_C_Receptacle_USB2.0_14P, SW1 Button, SW2 Button, U1 ESP32-C6-MINI-1

Commit message: crc v1
board finished and ready for assembly setup!
Connections:
- net GND: no longer U1.12 (IO0), U1.13 (IO1)
- no-connect marks 12 -> 14
Changed lines of the file:
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@@
 	)
 	(junction
-		(at 179.07 54.61)
-		(diameter 0)
-		(color 0 0 0 0)
-	)
-	(junction
 		(at 62.23 139.7)
 		(diameter 0)
@@
 	)
 	(no_connect
+		(at 179.07 57.15)
+	)
+	(no_connect
 		(at 209.55 72.39)
 	)
@@
 	)
 	(no_connect
+		(at 179.07 54.61)
+	)
+	(no_connect
 		(at 209.55 64.77)
 	)
@@
 	(wire
 		(pts
-			(xy 179.07 54.61) (xy 179.07 57.15)
-		)
-		(stroke
-			(width 0)
-			(type default)
-		)
-	)
-	(wire
-		(pts
 			(xy 66.04 115.57) (xy 66.04 114.3)
 		)
@@
 	(wire
 		(pts
-			(xy 179.07 52.07) (xy 173.99 52.07)
-		)
-		(stroke
-			(width 0)
-			(type default)
-		)
-	)
-	(wire
-		(pts
 			(xy 53.34 111.76) (xy 66.04 111.76)
 		)
@@
 	(wire
 		(pts
-			(xy 179.07 54.61) (xy 179.07 52.07)
-		)
-		(stroke
-			(width 0)
-			(type default)
-		)
-	)
-	(wire
-		(pts
 			(xy 53.34 142.24) (xy 62.23 142.24)
 		)
@@
 					(unit 1)
 				)
-			)
-		)
-	)
-	(symbol
-		(lib_id "power:GND")
-		(at 173.99 52.07 0)
-		(unit 1)
-		(exclude_from_sim no)
-		(in_bom yes)
-		(on_board yes)
-		(dnp no)
-		(property "Reference" "#PWR050"
-			(at 173.99 58.42 0)
-			(effects
-				(font
-					(size 1.27 1.27)
-				)
-				(hide yes)
-			)
-		)
-		(property "Value" "GND"
-			(at 173.99 55.88 0)
-			(effects
-				(font
-					(size 1.27 1.27)
-				)
-			)
-		)
-		(property "Footprint" ""
-			(at 173.99 52.07 0)
-			(effects
-				(font
-					(size 1.27 1.27)
-				)
-				(hide yes)
-			)
-		)
-		(property "Datasheet" ""
-			(at 173.99 52.07 0)
-			(effects
-				(font
-					(size 1.27 1.27)
-				)
-				(hide yes)
-			)
-		)
-		(property "Description" "Power symbol creates a global label with name \"GND\" , ground"
-			(at 173.99 52.07 0)
-			(effects
-				(font
-					(size 1.27 1.27)
-				)
-				(hide yes)
-			)
-		)
-		(pin "1"
-		)
-		(instances
-			(project "RC-W25"
-				(path "/427b2895-e3a6-4096-b101-5f65a3f7473e/01bd870e-4674-4257-9660-564635d632de"
-					(reference "#PWR050")
-					(unit 1)
-				)

Commit message: crc v1
quick fixes
Parts:
- R2, R4: value 5.7k -> 5.1k; LCSC# C852861 -> C490833

Commit message: crc v2
remote and receiver complete! assembly and orders have been prepared for purchasing.
Parts:
- C1, C2, C3, C4: LCSC# C338067 -> C12530; MPN (none) -> C12530
- C5, C6, C7, C9: LCSC# C22435938 -> C1525; MPN (none) -> C1525
- C8: LCSC# C380337 -> C87997; MPN (none) -> C87997
- D1, D2, D3: footprint Diode_SMD:D_0402_1005Metric -> footprints:D_0402_1005Metric; MPN (none) -> C316043
- DS1: footprint Library:FPC_30 -> footprints:FPC-30P-0.5mm; MPN (none) -> C2856808
- J1: MPN (none) -> C165948
- R1, R3, R6: MPN (none) -> C317921
- R2, R4: MPN (none) -> C490833
- R5: MPN (none) -> C861364
- R7: renamed from R8; MPN (none) -> C190095
- R8: renamed from R7; MPN (none) -> C190095
- SW1, SW2: MPN (none) -> C720477
- U1: LCSC# (none) -> C5736265; MPN (none) -> C5736265

Commit message: Custom RC V2
Final Remote + Receiver!

Special thanks to the CRCW25 Electrical Team who contributed to its development!

Jun
Katie
Nelson
David
Connections:
- net GPIO_RUMBLE_CNTL: now also U1.13 (IO1); no longer U1.15 (IO6)
- net SCL_DISPLAY: now also U1.16 (IO7)
- net SDA_DISPLAY: now also U1.15 (IO6)
- no-connect marks 14 -> 12
Other:
- moved on the sheet: R7
