File: RC-W25/RC_Motor&HallEffect.kicad_sch (KiCad schematic)
At the start: 9 parts, among them P2 JST CONN, Q1 NMOS, SW4 Button, U4 TMAG5253

Commit message: crc v2
remote and receiver complete! assembly and orders have been prepared for purchasing.
Parts:
- C16, C17: LCSC# C22435938 -> C1525; MPN (none) -> C1525
- D5: LCSC# C41376455 -> C64885; MPN (none) -> C64885
- P2: MPN (none) -> C3029440
- Q1: MPN (none) -> C443825
- R15, R16: MPN (none) -> C190095
- SW4: MPN (none) -> C720477
- U4: MPN (none) -> C22445458
Changed lines of the file:
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@@
+			)
+		)
+		(property "MPN" "C190095"
+			(at 152.4 67.31 0)
+			(effects
+				(font
+					(size 1.27 1.27)
+				)
+				(hide yes)
 			)
 		)
@@
 			)
 		)
-		(property "Datasheet" "https://www.lcsc.com/datasheet/lcsc_datasheet_2405231405_HRE-CGA0402X7R104K6R3GT_C22435938.pdf"
+		(property "Datasheet" ""
 			(at 76.2 119.38 0)
 			(effects
@@
 			)
 		)
-		(property "LCSC#" "C22435938"
+		(property "LCSC#" "C1525"
+			(at 76.2 119.38 0)
+			(effects
+				(font
+					(size 1.27 1.27)
+				)
+				(hide yes)
+			)
+		)
+		(property "MPN" "C1525"
 			(at 76.2 119.38 0)
 			(effects
@@
 		)
 		(property "LCSC#" "C720477"
+			(at 152.4 77.47 0)
+			(effects
+				(font
+					(size 1.27 1.27)
+				)
+				(hide yes)
+			)
+		)
+		(property "MPN" "C720477"
 			(at 152.4 77.47 0)
 			(effects
@@
 			)
 		)
+		(property "MPN" "C3029440"
+			(at 76.2 59.69 0)
+			(effects
+				(font
+					(size 1.27 1.27)
+				)
+				(hide yes)
+			)
+		)
 		(pin "1"
 		)
@@
 			)
 		)
+		(property "MPN" "C22445458 "
+			(at 93.98 113.03 0)
+			(effects
+				(font
+					(size 1.27 1.27)
+				)
+				(hide yes)
+			)
+		)
 		(pin "4"
 		)
@@
 		)
 		(property "LCSC#" "C190095"
+			(at 161.29 71.12 0)
+			(effects
+				(font
+					(size 1.27 1.27)
+				)
+				(hide yes)
+			)
+		)
+		(property "MPN" "C190095"
 			(at 161.29 71.12 0)
 			(effects
@@
 			)
 		)
-		(property "Datasheet" "https://www.lcsc.com/datasheet/lcsc_datasheet_2411011349_PIELENST-1N5819W-L_C41376455.pdf"
+		(property "Datasheet" ""
 			(at 85.09 60.96 0)
 			(effects
@@
 			)
 		)
-		(property "LCSC#" "C41376455"
+		(property "LCSC#" "C64885"
+			(at 85.09 60.96 0)
+			(effects
+				(font
+					(size 1.27 1.27)
+				)
+				(hide yes)
+			)
+		)
+		(property "MPN" "C64885"
 			(at 85.09 60.96 0)
 			(effects
@@
 			)
 		)
-		(property "Datasheet" "https://www.lcsc.com/datasheet/lcsc_datasheet_2405231405_HRE-CGA0402X7R104K6R3GT_C22435938.pdf"
+		(property "Datasheet" ""
 			(at 166.37 74.93 0)
 			(effects
@@
 			)
 		)
-		(property "LCSC#" "C22435938"
+		(property "LCSC#" "C1525"
+			(at 166.37 74.93 0)
+			(effects
+				(font
+					(size 1.27 1.27)
+				)
+				(hide yes)
+			)
+		)
+		(property "MPN" "C1525"
 			(at 166.37 74.93 0)
 			(effects
@@
 			(at 83.82 78.74 0)
 			(effects
+				(font
+					(size 1.27 1.27)
+				)
+				(hide yes)
+			)
+		)
+		(property "MPN" "C443825"
+			(at 83.82 78.74 0)
+			(effects
