File: remote/RC-W25.kicad_sch (KiCad schematic)
At the start: 0 parts

Commit message: CRC V3
V 3.0.0
Initial version of CRC V3, fully redesigned remote
Other:
- sheet RC_Battery renamed Power
- sheet RC_Connections renamed Connections
- sheet RC_Motor&HallEffect renamed Peripherals
Changed lines of the file:
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@@
 			(color 255 255 194 1.0000)
 		)
-		(property "Sheetname" "RC_Connections"
+		(property "Sheetname" "Connections"
 			(at 90.17 61.5184 0)
 			(effects
@@
 			(color 255 255 194 1.0000)
 		)
-		(property "Sheetname" "RC_Motor&HallEffect"
+		(property "Sheetname" "Peripherals"
 			(at 124.46 107.2384 0)
 			(effects
@@
 			(color 255 255 194 1.0000)
 		)
-		(property "Sheetname" "RC_Battery"
+		(property "Sheetname" "Power"
 			(at 160.02 61.5184 0)
 			(effects
