File: remote/RC_Connections.kicad_sch (KiCad schematic)
At the start: 28 parts, among them J1 USB_C_Receptacle_USB2.0_14P, SW1 Button, SW2 Button, U1 ESP32-C6-MINI-1

Commit message: CRC V3
V 3.0.0
Initial version of CRC V3, fully redesigned remote
Parts:
- removed H3: MountingHole, MountingHole:MountingHole_3.2mm_M3, symbol Mechanical:MountingHole
- removed R5: 390k, Resistor_SMD:R_0603_1608Metric, symbol Device:R_Small_US
- removed R6: 4.7k, Resistor_SMD:R_0402_1005Metric, symbol Device:R_Small_US
- added D4: RLED, Diode_SMD:D_0402_1005Metric_Pad0.77x0.64mm_HandSolder, symbol Device:LED_Small
- added D5: ORLED, Diode_SMD:D_0402_1005Metric_Pad0.77x0.64mm_HandSolder, symbol Device:LED_Small
- added D6: GLED, Diode_SMD:D_0402_1005Metric_Pad0.77x0.64mm_HandSolder, symbol Device:LED_Small
- added R10, R11, R9: 300, Resistor_SMD:R_0402_1005Metric_Pad0.72x0.64mm_HandSolder, symbol Device:R_Small_US
- added R2, R4: 4.7k, Resistor_SMD:R_0402_1005Metric_Pad0.72x0.64mm_HandSolder, symbol Device:R_Small_US
- added TP1, TP2, TP3: TEST POINT, TestPoint:TestPoint_Pad_2.0x2.0mm, symbol Connector:TestPoint
- C1: value 2.2uF -> 4.7uF; footprint Capacitor_SMD:C_0402_1005Metric -> Capacitor_SMD:C_0402_1005Metric_Pad0.74x0.62mm_HandSolder
- C2: value 2.2uF -> 10uF; footprint Capacitor_SMD:C_0402_1005Metric -> Capacitor_SMD:C_0402_1005Metric_Pad0.74x0.62mm_HandSolder
- C3, C4, C5, C9: footprint Capacitor_SMD:C_0402_1005Metric -> Capacitor_SMD:C_0402_1005Metric_Pad0.74x0.62mm_HandSolder
- C6: renamed from C7; footprint Capacitor_SMD:C_0402_1005Metric -> Capacitor_SMD:C_0402_1005Metric_Pad0.74x0.62mm_HandSolder
- C7: renamed from C6; footprint Capacitor_SMD:C_0402_1005Metric -> Capacitor_SMD:C_0402_1005Metric_Pad0.74x0.62mm_HandSolder
- C8: footprint Capacitor_SMD:C_0805_2012Metric -> Capacitor_SMD:C_0805_2012Metric_Pad1.18x1.45mm_HandSolder
- D1, D2, D3: footprint footprints:D_0402_1005Metric -> Diode_SMD:D_0402_1005Metric_Pad0.77x0.64mm_HandSolder
- DS1: value FPC 0.5mm 30P -> FPC 0.7mm 30P; footprint footprints:FPC-30P-0.5mm -> footprints:FPC 0.7mm 30P
- R1: value 4.7k -> 390k; footprint Resistor_SMD:R_0402_1005Metric -> Resistor_SMD:R_0603_1608Metric_Pad0.98x0.95mm_HandSolder; LCSC# C317921 -> C861364; MPN C317921 -> C861364
- R3, R7, R8: footprint Resistor_SMD:R_0402_1005Metric -> Resistor_SMD:R_0402_1005Metric_Pad0.72x0.64mm_HandSolder
- R5: renamed from R2; footprint Resistor_SMD:R_0402_1005Metric -> Resistor_SMD:R_0402_1005Metric_Pad0.72x0.64mm_HandSolder
- R6: renamed from R4; footprint Resistor_SMD:R_0402_1005Metric -> Resistor_SMD:R_0402_1005Metric_Pad0.72x0.64mm_HandSolder
Connections:
- net +3.3V: now also R2.1, R4.1; no longer R1.1
- net +USB5V: now also TP1.1
- net GND: now also R1.2, R10.2, R11.2, R9.2; no longer DS1.7 (N.C.)
- net GPIO_MODE: now also U1.10 (IO5); no longer U1.9 (IO4)
- net SCL_DISPLAY: now also DS1.20 (D2), U1.25 (IO19), R4.2, TP3.1; no longer U1.16 (IO7)
- net SDA_DISPLAY: now also U1.26 (IO20), R2.2, TP2.1; no longer R3.2, U1.15 (IO6)
- net at DS1.14 (Reset): now also R3.2; no longer R1.2
- net at DS1.26 (IREF): now also R1.1
- net at DS1.27 (VCOMH): now also C1.1; no longer C2.1
- net at DS1.28 (VDisplay): now also C2.1; no longer C1.1
- net CHSTAT1: now reaches U1.24 (IO18)
- net at U1.27 (IO21): now also D4.2 (A)
- net at U1.29 (IO23): now also D6.2 (A)
- net ADC_HALLEFFECT1 renamed ADC_JOYSTICK
- net GPIO_EN1: no longer names the net of U1.28 (IO22)
- net GPIO_EN1: now also D5.2 (A)
- new net: D6.1 (K), R11.1
- new net: D5.1 (K), R10.1
- new net: D4.1 (K), R9.1
- new net CHSTAT2: U1.16 (IO7)
- new net CH_EN: U1.15 (IO6)
- new net ON/OFF: U1.9 (IO4)
- no-connect marks 12 -> 6
Other:
- note added: "OLED Display"
- note removed: "Differential Routing"
- note removed: "SSD1306 I2C"
- moved on the sheet: C5, C6, C7, C8, C9, D1, D2, D3, H1, H2, J1, R5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

Commit message: Finalized design for review and order
Parts:
- DS1: value FPC 0.7mm 30P -> FPC 30P; footprint footprints:FPC 0.7mm 30P -> footprints:FPC-30P-0.5mm
Connections:
- net SCL_DISPLAY: now also U1.26 (IO20); no longer U1.25 (IO19)
- net SDA_DISPLAY: now also U1.25 (IO19); no longer U1.26 (IO20)
Other:
- moved on the sheet: TP2, TP3
Changed lines of the file:
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@@
 	)
 	(junction
-		(at 256.54 72.39)
-		(diameter 0)
-		(color 0 0 0 0)
-	)
-	(junction
 		(at 275.59 77.47)
 		(diameter 0)
@@
 	)
 	(junction
-		(at 259.08 69.85)
+		(at 135.89 55.88)
 		(diameter 0)
 		(color 0 0 0 0)
 	)
 	(junction
-		(at 135.89 55.88)
+		(at 146.05 48.26)
 		(diameter 0)
 		(color 0 0 0 0)
 	)
 	(junction
-		(at 146.05 48.26)
+		(at 260.35 69.85)
 		(diameter 0)
 		(color 0 0 0 0)
@@
 	)
 	(junction
+		(at 256.54 72.39)
+		(diameter 0)
+		(color 0 0 0 0)
+	)
+	(junction
 		(at 275.59 80.01)
 		(diameter 0)
@@
 	(wire
 		(pts
+			(xy 260.35 69.85) (xy 269.24 69.85)
+		)
+		(stroke
+			(width 0)
+			(type default)
+		)
+	)
+	(wire
+		(pts
 			(xy 193.04 72.39) (xy 222.25 72.39)
 		)
@@
 	(wire
 		(pts
-			(xy 269.24 69.85) (xy 259.08 69.85)
-		)
-		(stroke
-			(width 0)
-			(type default)
-		)
-	)
-	(wire
-		(pts
-			(xy 256.54 72.39) (xy 269.24 72.39)
-		)
-		(stroke
-			(width 0)
-			(type default)
-		)
-	)
-	(wire
-		(pts
 			(xy 252.73 72.39) (xy 256.54 72.39)
 		)
@@
 	(wire
 		(pts
-			(xy 259.08 69.85) (xy 252.73 69.85)
+			(xy 38.1 170.18) (xy 35.56 170.18)
 		)
 		(stroke
@@
 	(wire
 		(pts
-			(xy 38.1 170.18) (xy 35.56 170.18)
+			(xy 212.09 54.61) (xy 222.25 54.61)
 		)
 		(stroke
@@
 	(wire
 		(pts
-			(xy 212.09 54.61) (xy 222.25 54.61)
+			(xy 35.56 99.06) (xy 57.15 99.06)
 		)
 		(stroke
@@
 	(wire
 		(pts
-			(xy 35.56 99.06) (xy 57.15 99.06)
+			(xy 45.72 33.02) (xy 35.56 33.02)
 		)
 		(stroke
@@
 	(wire
 		(pts
-			(xy 45.72 33.02) (xy 35.56 33.02)
+			(xy 35.56 73.66) (xy 57.15 73.66)
 		)
 		(stroke
@@
 	(wire
 		(pts
-			(xy 35.56 73.66) (xy 57.15 73.66)
+			(xy 45.72 93.98) (xy 35.56 93.98)
 		)
 		(stroke
@@
 	(wire
 		(pts
-			(xy 45.72 93.98) (xy 35.56 93.98)
+			(xy 252.73 69.85) (xy 260.35 69.85)
 		)
 		(stroke
@@
 	(wire
 		(pts
+			(xy 256.54 72.39) (xy 269.24 72.39)
+		)
+		(stroke
+			(width 0)
+			(type default)
+		)
+	)
+	(wire
+		(pts
 			(xy 45.72 48.26) (xy 35.56 48.26)
 		)
@@
 		)
 	)
-	(global_label "GPIO_MODE"
+	(global_label "SCL_DISPLAY"
 		(shape input)
-		(at 212.09 64.77 180)
+		(at 269.24 72.39 0)
 		(fields_autoplaced yes)
 		(effects
@@
 				(size 1.27 1.27)
 			)
-			(justify right)
+			(justify left)
 		)
 		(property "Intersheetrefs" "${INTERSHEET_REFS}"
-			(at 198.461 64.77 0)
+			(at 284.26 72.39 0)
 			(effects
 				(font
 					(size 1.27 1.27)
 				)
-				(justify right)
+				(justify left)
 				(hide yes)
 			)
 		)
 	)
-	(global_label "SCL_DISPLAY"
+	(global_label "GPIO_MODE"
 		(shape input)
-		(at 269.24 69.85 0)
+		(at 212.09 64.77 180)
 		(fields_autoplaced yes)
 		(effects
@@
 				(size 1.27 1.27)
 			)
-			(justify left)
+			(justify right)
 		)
 		(property "Intersheetrefs" "${INTERSHEET_REFS}"
-			(at 284.26 69.85 0)
+			(at 198.461 64.77 0)
 			(effects
 				(font
 					(size 1.27 1.27)
 				)
-				(justify left)
+				(justify right)
 				(hide yes)
 			)
@@
 	(global_label "SDA_DISPLAY"
 		(shape input)
-		(at 64.77 119.38 0)
+		(at 269.24 69.85 0)
 		(fields_autoplaced yes)
 		(effects
@@
 		)
 		(property "Intersheetrefs" "${INTERSHEET_REFS}"
-			(at 79.8505 119.38 0)
+			(at 284.3205 69.85 0)
 			(effects
 				(font
@@
 		)
 	)
-	(global_label "USB_D-"
+	(global_label "SDA_DISPLAY"
 		(shape input)
-		(at 163.83 48.26 0)
+		(at 64.77 119.38 0)
 		(fields_autoplaced yes)
 		(effects
@@
 		)
 		(property "Intersheetrefs" "${INTERSHEET_REFS}"
-			(at 174.4352 48.26 0)
+			(at 79.8505 119.38 0)
 			(effects
 				(font
@@
 		)
 	)
-	(global_label "ADC_BATTERYPERCENT"
+	(global_label "USB_D-"
 		(shape input)
-		(at 212.09 59.69 180)
+		(at 163.83 48.26 0)
 		(fields_autoplaced yes)
 		(effects
@@
 				(size 1.27 1.27)
 			)
-			(justify right)
+			(justify left)
 		)
 		(property "Intersheetrefs" "${INTERSHEET_REFS}"
-			(at 188.3011 59.69 0)
+			(at 174.4352 48.26 0)
 			(effects
 				(font
 					(size 1.27 1.27)
 				)
-				(justify right)
+				(justify left)
 				(hide yes)
 			)
 		)
 	)
-	(global_label "USB_D-"
+	(global_label "ADC_BATTERYPERCENT"
 		(shape input)
-		(at 255.27 54.61 0)
+		(at 212.09 59.69 180)
 		(fields_autoplaced yes)
 		(effects
@@
 				(size 1.27 1.27)
 			)
-			(justify left)
+			(justify right)
 		)
 		(property "Intersheetrefs" "${INTERSHEET_REFS}"
-			(at 265.8752 54.61 0)
+			(at 188.3011 59.69 0)
 			(effects
 				(font
 					(size 1.27 1.27)
 				)
-				(justify left)
+				(justify right)
 				(hide yes)
 			)
 		)
 	)
-	(global_label "SDA_DISPLAY"
+	(global_label "USB_D-"
 		(shape input)
-		(at 269.24 72.39 0)
+		(at 255.27 54.61 0)
 		(fields_autoplaced yes)
 		(effects
@@
 		)
 		(property "Intersheetrefs" "${INTERSHEET_REFS}"
-			(at 284.3205 72.39 0)
+			(at 265.8752 54.61 0)
 			(effects
 				(font
@@
 	(symbol
 		(lib_id "Connector:TestPoint")
-		(at 259.08 69.85 0)
+		(at 256.54 72.39 0)
 		(mirror y)
 		(unit 1)
@@
 		(dnp no)
 		(property "Reference" "TP3"
-			(at 263.398 66.548 0)
+			(at 256.286 71.374 0)
 			(effects
 				(font
@@
 		)
 		(property "Value" "TEST POINT"
-			(at 267.208 68.072 0)
+			(at 264.414 71.628 0)
 			(effects
 				(font
@@
 		)
 		(property "Footprint" "TestPoint:TestPoint_Pad_2.0x2.0mm"
-			(at 254 69.85 0)
+			(at 251.46 72.39 0)
 			(effects
 				(font
@@
 		)
 		(property "Datasheet" "https://www.koaspeer.com/pdfs/RC.pdf"
-			(at 254 69.85 0)
+			(at 251.46 72.39 0)
 			(effects
 				(font
@@
 		)
 		(property "Description" "test point"
-			(at 259.08 69.85 0)
+			(at 256.54 72.39 0)
 			(effects
 				(font
@@
 		)
 		(property "Manufacturer" ""
-			(at 259.08 69.85 0)
+			(at 256.54 72.39 0)
 			(effects
 				(font
@@
 		)
 		(property "Manufacturer Part" ""
-			(at 259.08 69.85 0)
+			(at 256.54 72.39 0)
 			(effects
 				(font
@@
 		)
 		(property "Supplier" ""
-			(at 259.08 69.85 0)
+			(at 256.54 72.39 0)
 			(effects
 				(font
@@
 		)
 		(property "Supplier Part" ""
-			(at 259.08 69.85 0)
+			(at 256.54 72.39 0)
 			(effects
 				(font
@@
 			)
 		)
-		(property "Value" "FPC 0.7mm 30P"
+		(property "Value" "FPC 30P"
 			(at 27.94 29.718 0)
 			(effects
@@
 			)
 		)
-		(property "Footprint" "footprints:FPC 0.7mm 30P"
+		(property "Footprint" "footprints:FPC-30P-0.5mm"
 			(at 27.94 104.14 0)
 			(effects
@@
 	(symbol
 		(lib_id "Connector:TestPoint")
-		(at 256.54 72.39 0)
+		(at 260.35 69.85 0)
 		(mirror y)
 		(unit 1)
@@
 		(dnp no)
 		(property "Reference" "TP2"
-			(at 256.032 71.374 0)
+			(at 264.922 66.294 0)
 			(effects
 				(font
@@
 		)
 		(property "Value" "TEST POINT"
-			(at 264.16 71.628 0)
+			(at 268.478 68.326 0)
 			(effects
 				(font
@@
 		)
 		(property "Footprint" "TestPoint:TestPoint_Pad_2.0x2.0mm"
-			(at 251.46 72.39 0)
+			(at 255.27 69.85 0)
 			(effects
 				(font
@@
 		)
 		(property "Datasheet" "https://www.koaspeer.com/pdfs/RC.pdf"
-			(at 251.46 72.39 0)
+			(at 255.27 69.85 0)
 			(effects
 				(font
@@
 		)
 		(property "Description" "test point"
-			(at 256.54 72.39 0)
+			(at 260.35 69.85 0)
 			(effects
 				(font
@@
 		)
 		(property "Manufacturer" ""
-			(at 256.54 72.39 0)
+			(at 260.35 69.85 0)
 			(effects
 				(font
@@
 		)
 		(property "Manufacturer Part" ""
-			(at 256.54 72.39 0)
+			(at 260.35 69.85 0)
 			(effects
 				(font
@@
 		)
 		(property "Supplier" ""
-			(at 256.54 72.39 0)
+			(at 260.35 69.85 0)
 			(effects
 				(font
@@
 		)
 		(property "Supplier Part" ""
-			(at 256.54 72.39 0)
+			(at 260.35 69.85 0)
 			(effects
 				(font
